Commit message: edit: readme; update instructions/list of compatible packages

File: workstation_description/workstation_model.urdf.xacro (robot description, xacro)
@@ -13,5 +13,5 @@
     xmlns:physics="http://playerstage.sourceforge.net/gazebo/xmlschema/#physics"
     xmlns:xacro="http://ros.org/wiki/xacro">
-  <xacro:macro name="workstation" params="prefix">
+  <xacro:macro name="workstation" params="prefix namespace">
   <xacro:include filename="$(find uml_hri_nerve_armada_workstation)/workstation_gazebo/workstation_model_gazebo.xacro" />
   <xacro:include filename="$(find uml_hri_nerve_armada_workstation)/workstation_gazebo/workstation_depth_cameras_gazebo.xacro" />
@@ -70,9 +70,9 @@
     <origin xyz="0.0 0.0 0.0" rpy="${-pi/2} 0.0 ${-pi/2}" />
     <parent link="${prefix}top_camera_link" />
-    <child link="${prefix}top_optical" />
+    <child link="${namespace}/${prefix}top_optical" />
     <axis xyz="0 0 0" />
   </joint>
   <!-- TOP OPTICAL -->
-  <link name="${prefix}top_optical" />
+  <link name="${namespace}/${prefix}top_optical" />
   <!-- TABLE TO PEDESTAL JOINT -->
   <joint name="table_to_pedestal_joint" type="fixed">
@@ -230,9 +230,9 @@
     <origin xyz="0.0 0.0 0.0" rpy="${-pi/2} 0.0 ${-pi/2}" />
     <parent link="${prefix}left_camera_link" />
-    <child link="${prefix}left_optical" />
+    <child link="${namespace}/${prefix}left_optical" />
     <axis xyz="0 0 0" />
   </joint>
   <!-- LEFT OPTICAL -->
-  <link name="${prefix}left_optical" />
+  <link name="${namespace}/${prefix}left_optical" />
   <!-- TABLE TO RIGHT HORIZONTAL ARM JOINT -->
   <joint name="table_to_right_horizontal_arm_joint" type="fixed">
@@ -334,9 +334,9 @@
     <origin xyz="0.0 0.0 0.0" rpy="${-pi/2} 0.0 ${-pi/2}" />
     <parent link="${prefix}right_camera_link" />
-    <child link="${prefix}right_optical" />
+    <child link="${namespace}/${prefix}right_optical" />
     <axis xyz="0 0 0" />
   </joint>
   <!-- RIGHT OPTICAL -->
-  <link name="${prefix}right_optical" />
+  <link name="${namespace}/${prefix}right_optical" />
   <!-- TABLE TO REAR HORIZONTAL ARM JOINT -->
   <joint name="table_to_rear_horizontal_arm_joint" type="fixed">
@@ -434,9 +434,9 @@
     <origin xyz="0.0 0.0 0.0" rpy="${-pi/2} 0.0 ${-pi/2}" /> <!-- X=Z, -Y=Y, Z=X-->
     <parent link="${prefix}rear_camera_link" />
-    <child link="${prefix}rear_optical" />
+    <child link="${namespace}/${prefix}rear_optical" />
     <axis xyz="0 0 0" />
   </joint>
   <!-- REAR OPTICAL -->
-  <link name="${prefix}rear_optical" />
+  <link name="${namespace}/${prefix}rear_optical" />
   </xacro:macro>
 </robot>

File: workstation_description/workstation_model_macro.urdf.xacro (robot description, xacro)
@@ -14,5 +14,5 @@
     xmlns:xacro="http://ros.org/wiki/xacro" name="ur5e_d435_millibar_combined_r2f85" >
   <xacro:include filename="$(find uml_hri_nerve_armada_workstation)/workstation_description/workstation_model.urdf.xacro" />
-  <xacro:workstation prefix="table_"/>
+  <xacro:workstation prefix="table_" namespace=""/>
   <!-- This is not required because the "world" link already exists
   <link name="world" />
